File: PCB/new_PCB/new_PCB/new_PCB.kicad_sch (KiCad schematic)
At the start: 18 parts, among them J1 XT60PW-F, J2 XT60PW-F, J3 MOLEX-Connector, J4 MOLEX-Connector, J5 MOLEX-Connector, J6 MOLEX-Connector, J7 MOLEX-Connector, J8 MOLEX-Connector, U1 ESP32-S3-DEVKITC-1-N16R8V

Commit message: Add changes to new pcb
Parts:
- added H1, H2, H3, H4: MountingHole, MountingHole:MountingHole_3.2mm_M3_ISO14580, symbol Mechanical:MountingHole
Connections:
- net RX2: now also U1.J1_4 (GPIO4); no longer U1.J1_5 (GPIO5)
- net TX2: now also U1.J1_5 (GPIO5); no longer U1.J1_4 (GPIO4)

Commit message: Final PCB version
Parts:
- added C1, C3: 100nF, Capacitor_SMD:C_0805_2012Metric, symbol Device:C
- added C2: 100uF, Capacitor_THT:CP_Radial_D6.3mm_P2.50mm, symbol Device:C
- added Q1, Q2: Q_PMOS, Package_TO_SOT_SMD:TO-252-2, symbol Device:Q_PMOS
- added R10, R11: 10k, Resistor_SMD:R_0805_2012Metric_Pad1.20x1.40mm_HandSolder, symbol Device:R
- added R7: 100k, Resistor_SMD:R_0805_2012Metric_Pad1.20x1.40mm_HandSolder, symbol Device:R
- added R8: 22k, Resistor_SMD:R_0805_2012Metric_Pad1.20x1.40mm_HandSolder, symbol Device:R
- added R9: 1k, Resistor_SMD:R_0805_2012Metric_Pad1.20x1.40mm_HandSolder, symbol Device:R
Connections:
- net GND: now also C1.2, C2.2, C3.2, R10.2, R11.2, R8.2
- net BAT_LVL: now reaches U1.J3_18 (GPIO21)
- net BAT_LVL: now also R9.2
- removed net VBUS: J1.1 (P), J2.1 (P), J3.2, J4.2, J5.2, J6.2, J7.2, J8.2, U2.8 (IN+)
- new net: Q1.1 (G), R10.1
- new net: Q2.1 (G), R11.1
- new net: C1.1, R7.2, R8.1, R9.1
- new net VBAT: J1.1 (P), J2.1 (P), Q1.3 (S), Q2.3 (S)
- new net VBUS_1: J6.2, J7.2, J8.2, Q1.2 (D), R7.1
- new net VBUS_2: C2.1, C3.1, J3.2, J4.2, J5.2, Q2.2 (D), U2.8 (IN+)
Other:
- moved on the sheet: U2
